File: hardware/MG2639 Cellular Shield.sch (EAGLE design)
At the start: 54 parts, among them J1 SIMHOLDER, J2 ARDUINO_R3_SHIELD, Q1 MMBT2222A, U1 SPX29302, U3 MG2639V3

Commit message: Adding stand-off holes. Moving GPS UART to pins 8/9 (better support for faster buad rates). Adding jumpers to select hardware UART for GPS too.
Parts:
- added JP7: USB, SparkFun-Connectors:M05PTH
- added SJ10, SJ7, SJ9: JUMPER-PAD-3-2OF3_NC_BY_TRACE, SparkFun-Passives:JUMPER-PAD-3-2OF3_NC_BY_TRACE
- added SJ8: FTDI_VCCIO, SparkFun-Passives:JUMPER-PAD-2-NOYES_SILK
- added STANDOFF1, STANDOFF2, STANDOFF3, STANDOFF4: STAND-OFF, SparkFun-Electromechanical:STAND-OFF
- JP2: value AUDIO -> M02PTH; device SparkFun-Connectors:M07 -> SparkFun-Connectors:M02PTH
- JP3: value FTDI_BASICPTH -> AUDIO; device SparkFun-Connectors:FTDI_BASICPTH -> SparkFun-Connectors:M07
- JP4: value (none) -> FTDI_BASICPTH; device SparkFun-Connectors:M07 -> SparkFun-Connectors:FTDI_BASICPTH
- JP5: value (none) -> MISC
- JP6: value M02PTH -> UART2
- SJ1: value JUMPER-PAD-2-NC_BY_TRACE -> BOOT; device SparkFun-Passives:JUMPER-PAD-2-NC_BY_TRACE -> SparkFun-Passives:JUMPER-PAD-3-2OF3_NC_BY_TRACE
- SJ2: value JUMPER-PAD-2-NC_BY_TRACE -> VBAT1
- SJ3: value JUMPER-PAD-3-2OF3_NC_BY_TRACE -> VBAT_EN; device SparkFun-Passives:JUMPER-PAD-3-2OF3_NC_BY_TRACE -> SparkFun-Passives:JUMPER-PAD-2-NOYES_SILK
- SJ4: value JUMPER-PAD-3-2OF3_NC_BY_TRACE -> JUMPER-PAD-2-NC_BY_TRACE; device SparkFun-Passives:JUMPER-PAD-3-2OF3_NC_BY_TRACE -> SparkFun-Passives:JUMPER-PAD-2-NC_BY_TRACE
Connections:
- new net GRX-SOFT: J2.*D9, SJ10.3
- new net GTX-SOFT: J2.D8, SJ9.3
- new net N$11: JP4.4, SJ8.1
- new net N$12: JP1.2, JP2.2, SJ3.2
- net !SYSRST: now also JP5.5; no longer JP4.7
- net 3.3V: now also SJ5.3; no longer SJ4.3
- net 3.8V: now also SJ3.1, SJ4.1; no longer JP1.2, JP6.2, SJ1.1
- net 5V: now also SJ5.1; no longer SJ4.1
- net EAR_L: now also JP3.6; no longer JP2.6
- net GND: now also JP2.1, JP3.7, JP4.6, JP5.4, JP7.1; no longer JP2.7, JP3.6, JP4.4, JP5.1, JP6.1
- net GPIO1/SCL: now also JP5.1; no longer JP4.1
- net GPIO2/SDA: now also JP5.2; no longer JP4.2
- net GRX-HV: now also SJ10.2; no longer J2.D4
- net GTX-HV: now also SJ9.2; no longer J2.*D5
- net MIC_N0: now also JP3.1; no longer JP2.1
- net MIC_P0: now also JP3.2; no longer JP2.2
- net MIC_P1: now also JP3.3; no longer JP2.3
- net N$10: now also JP7.3; no longer JP5.3
- net N$2: now also JP7.4; no longer JP5.4
- net N$5: now also SJ1.2; no longer SJ3.2
- net N$6: now also SJ1.1; no longer SJ3.1
- net ON/OFF: now also SJ1.3; no longer SJ3.3
- net RECN: now also JP3.4; no longer JP2.4
- net RECP: now also JP3.5; no longer JP2.5
- net RX-HV: now also JP4.3, SJ6.2; no longer JP3.3, SJ5.2
- net RX-SOFT: now also J2.*D3; no longer J2.D2
- net RX2-2.8V: now also JP6.1; no longer JP4.6
- net RXI: now also SJ7.1, SJ9.1; no longer SJ6.1
- net TX-HV: now also JP4.2, SJ7.2; no longer JP3.2, SJ6.2
- net TX-SOFT: now also J2.D2, SJ7.3; no longer J2.*D3, SJ5.3
- net TX2-2.8V: now also JP6.2; no longer JP4.5
- net TXO: now also SJ10.1, SJ6.1; no longer SJ5.1
- net VCCB: now also SJ5.2, SJ8.2; no longer SJ4.2
- net VDDIO: now also JP5.3; no longer JP4.3
- net V_GPS: now also SJ4.2; no longer SJ1.2
Other:
- note added: "Cut SJ2 to power from battery"
- note added: "Input Voltage Range: 4.5-16V"
- note added: "Open SJ4 to disconnect GPS power from board power."
- note added: "Optional battery input. Input range: 3.4-4.2V To use battery, cut SJ2 and short SJ3."
- note added: "Power Requirements: Max current: 300mA Standby current: 24mA Talk current: 128mA"
- note added: "SJ1 selects between Arduino pin-control of !PWRKEY! or permanently turning module on during power-up."
- note added: "Select between hardware UART and software UART for both GPS and cellular UART's Both default to software"
- note added: "Short SJ3 to power from battery"
- note added: "Short SJ8 to enable FTDI VCC to power high- side of level shifter."
- note removed: "Cut to power from battery"
- note removed: "Open SJ1 to disconnect GPS power from board power."
- note removed: "Select between hardware UART and software UART Default = Software"
- moved on the sheet: C1, C6, C8, C9, D1, J2, JP1, JP5, JP6, R1, R10, R11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

Commit message: Defaulting TXB0104 HV to 5V. Fixing connector names. Adding measures.
Parts:
- removed J1: SIMHOLDER, SparkFun-Connectors:SIMHOLDERSIM
- removed J2: ARDUINO_R3_SHIELD, SparkFun-Boards:ARDUINO_R3_SHIELDNOLABELS
- added JP8: FTDI_BASICPTH, SparkFun-Connectors:FTDI_BASICPTH
- added JP9: USB, SparkFun-Connectors:M05PTH
- JP3: value AUDIO -> ARDUINO_R3_SHIELD; device SparkFun-Connectors:M07 -> SparkFun-Boards:ARDUINO_R3_SHIELDNOLABELS
- JP4: value FTDI_BASICPTH -> SIMHOLDER; device SparkFun-Connectors:FTDI_BASICPTH -> SparkFun-Connectors:SIMHOLDERSIM
- JP5: value MISC -> AUDIO; device SparkFun-Connectors:M05PTH -> SparkFun-Connectors:M07
- JP6: value UART2 -> MISC; device SparkFun-Connectors:M02PTH -> SparkFun-Connectors:M05PTH
- JP7: value USB -> UART2; device SparkFun-Connectors:M05PTH -> SparkFun-Connectors:M02PTH
- U2: value (none) -> TXB0104
Connections:
- new net JP9: JP3.D8
- net !SYSRST: now also JP6.5; no longer JP5.5
- net 3.3V: now also JP3.3.3V, SJ5.1; no longer J2.3.3V, SJ5.3
- net 5V: now also JP3.5V, SJ5.3; no longer J2.5V, SJ5.1
- net A1: now also JP3.A1; no longer J2.A1
- net A2: now also JP3.A2; no longer J2.A2
- net A3: now also JP3.A3; no longer J2.A3
- net A4: now also JP3.A4; no longer J2.A4
- net A5: now also JP3.A5; no longer J2.A5
- net CELL_RESET: now also JP3.*D6; no longer J2.*D6
- net EAR_L: now also JP5.6; no longer JP3.6
- net GND: now also JP3.GND@0, JP3.GND@1, JP3.GND@2, JP4.GND, JP5.7, JP6.4, JP8.6, JP9.1; no longer J1.GND, J2.GND@0, J2.GND@1, J2.GND@2, JP3.7, JP4.6, JP5.4, JP7.1
- net GPIO1/SCL: now also JP6.1; no longer JP5.1
- net GPIO2/SDA: now also JP6.2; no longer JP5.2
- net GRX-SOFT: now also JP3.*D9; no longer J2.*D9
- net GTX-SOFT: no longer J2.D8
- net MIC_N0: now also JP5.1; no longer JP3.1
- net MIC_P0: now also JP5.2; no longer JP3.2
- net MIC_P1: now also JP5.3; no longer JP3.3
- net N$10: now also JP9.3; no longer JP7.3
- net N$11: now also JP8.4; no longer JP4.4
- net N$2: now also JP9.4; no longer JP7.4
- net ON/OFF: now also JP3.D7; no longer J2.D7
- net RECN: now also JP5.4; no longer JP3.4
- net RECP: now also JP5.5; no longer JP3.5
- net RESET: now also JP3.RES; no longer J2.RES
- net RING: now also JP3.A0; no longer J2.A0
- net RX-HV: now also JP8.3; no longer JP4.3
- net RX-SOFT: now also JP3.*D3; no longer J2.*D3
- net RX2-2.8V: now also JP7.1; no longer JP6.1
- net RXI: now also JP3.RX; no longer J2.RX
- net SIM_CLK: now also JP4.CLK; no longer J1.CLK
- net SIM_DATA: now also JP4.I/O; no longer J1.I/O
- net SIM_RST: now also JP4.RST; no longer J1.RST
- net TX-HV: now also JP8.2; no longer JP4.2
- net TX-SOFT: now also JP3.D2; no longer J2.D2
- net TX2-2.8V: now also JP7.2; no longer JP6.2
- net TXO: now also JP3.TX; no longer J2.TX
- net VDDIO: now also JP6.3; no longer JP5.3
- net VRAW: now also JP3.VIN; no longer J2.VIN
- net VSIM: now also JP4.VCC, JP4.VPP; no longer J1.VCC, J1.VPP
Other:
- note added: "Select between 3.3V and 5V Default = 5V"
- note removed: "Select between 3.3V and 5V Default = 3.3V"
