File: Hardware/MG2639 Cellular Shield.brd (EAGLE design)
At the start: 53.3 x 74.9 mm, 64 parts, among them Q1 MMBT2222A, U1 SPX29302, U2 TXB0104, U3 MG2639V3

Commit message: Updating LiPo connector value to DNP
Parts:
- JP1: value LiPo -> DNP
