File: Hardware/MG2639 Cellular Shield.sch (EAGLE design)
At the start: 64 parts, among them Q1 MMBT2222A, U1 SPX29302, U2 TXB0104, U3 MG2639V3

Commit message: Updating LiPo connector value to DNP
Parts:
- JP1: value LiPo -> DNP
Changed lines of the file:
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@@
 <?xml version="1.0" encoding="utf-8"?>
 <!DOCTYPE eagle SYSTEM "eagle.dtd">
-<eagle version="7.1.0">
+<eagle version="7.5.0">
 <drawing>
 <settings>
@@
 <layer number="255" name="routoute" color="7" fill="1" visible="yes" active="yes"/>
 </layers>
-<schematic xreflabel="%F%N/%S.%C%R" xrefpart="/%S.%C%R">
+<schematic xreflabel="%F%N/%S" xrefpart="/%S.%C%R">
 <attributes>
 </attributes>
@@
 <part name="SJ2" library="SparkFun-Passives" deviceset="JUMPER-PAD-2-NC_BY_TRACE" device="" value="VBAT1"/>
 <part name="GND17" library="SparkFun1" deviceset="GND" device=""/>
-<part name="JP1" library="SparkFun-Connectors" deviceset="M02" device="JST-PTH-2" value="LiPo"/>
+<part name="JP1" library="SparkFun-Connectors" deviceset="M02" device="JST-PTH-2" value="DNP"/>
 <part name="JP9" library="SparkFun-Connectors" deviceset="M05" device="PTH" value="USB"/>
 <part name="SJ1" library="SparkFun-Passives" deviceset="JUMPER-PAD-3-2OF3_NC_BY_TRACE" device="" value="BOOT"/>
